File: HW/_autosave-AD5791 Linearity Calibrator.kicad_pcb (KiCad board)
At the start: 4 copper layers, 88 x 56 mm, 47 parts, among them J1 OUTPUT, J2 PWR, J4 REF, SW1 RST, U1 Pico, U11 7533, U12 ADuM1201AR, U2 AD5791BRUZ, U4 OPA189, U5 OPA189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

Commit message: NOMC network
Routing:
- added copper zone on B.Cu, net /3V3IN
- added copper zone on In1.Cu, net /3V3IN
- added copper zone on In2.Cu, net /3V3IN
- removed copper zone on B.Cu, net +15V
- removed copper zone on In1.Cu, net +15V
- removed copper zone on In2.Cu, net +15V
Changed lines of the file:
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@@
     )
   )
-  (zone (net 1) (net_name "+15V") (layers "In1.Cu" "In2.Cu" "B.Cu") (hatch edge 0.5)
+  (zone (net 59) (net_name "/3V3IN") (layers "In1.Cu" "In2.Cu" "B.Cu") (hatch edge 0.5)
     (priority 15)
     (connect_pads yes (clearance 0.127))
