File: HW/AD5791 Linearity Calibrator.kicad_sch (KiCad schematic)
At the start: 52 parts, among them J1 OUTPUT, J2 PWR, J3 REF, J4 REF, J5 REF, J6 REF, SW1 RST, U1 Pico, U11 7533, U12 ADuM1201AR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

Commit message: layout, copper edges
Parts:
- added J10, J7, J8, J9: Conn_01x01, Connector_PinHeader_2.54mm:PinHeader_1x01_P2.54mm_Vertical, symbol Connector_Generic:Conn_01x01
Connections:
- net GND: now also J10.1 (Pin_1), J7.1 (Pin_1), J8.1 (Pin_1), J9.1 (Pin_1)
Changed lines of the file:
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@@
   (junction (at 278.13 261.62) (diameter 0) (color 0 0 0 0)
   )
+  (junction (at 257.81 228.6) (diameter 0) (color 0 0 0 0)
+  )
   (junction (at 217.17 255.27) (diameter 0) (color 0 0 0 0)
   )
   (junction (at 59.69 80.01) (diameter 0) (color 0 0 0 0)
   )
+  (junction (at 257.81 238.76) (diameter 0) (color 0 0 0 0)
+  )
   (junction (at 223.52 45.72) (diameter 0) (color 0 0 0 0)
   )
@@
   (junction (at 365.76 208.28) (diameter 0) (color 0 0 0 0)
   )
+  (junction (at 257.81 233.68) (diameter 0) (color 0 0 0 0)
+  )
   (junction (at 213.36 45.72) (diameter 0) (color 0 0 0 0)
   )
@@
     (stroke (width 0) (type default))
   )
+  (wire (pts (xy 257.81 228.6) (xy 257.81 233.68))
+    (stroke (width 0) (type default))
+  )
   (wire (pts (xy 241.3 58.42) (xy 241.3 55.88))
     (stroke (width 0) (type default))
@@
     (stroke (width 0) (type default))
   )
+  (wire (pts (xy 257.81 223.52) (xy 257.81 228.6))
+    (stroke (width 0) (type default))
+  )
   (wire (pts (xy 327.66 195.58) (xy 325.12 195.58))
     (stroke (width 0) (type default))
@@
     (stroke (width 0) (type default))
   )
+  (wire (pts (xy 257.81 238.76) (xy 257.81 241.3))
+    (stroke (width 0) (type default))
+  )
   (wire (pts (xy 243.84 115.57) (xy 260.35 115.57))
     (stroke (width 0) (type default))
@@
     (stroke (width 0) (type default))
   )
+  (wire (pts (xy 255.27 233.68) (xy 257.81 233.68))
+    (stroke (width 0) (type default))
+  )
   (wire (pts (xy 81.915 58.42) (xy 93.345 58.42))
     (stroke (width 0) (type default))
@@
     (stroke (width 0) (type default))
   )
+  (wire (pts (xy 255.27 238.76) (xy 257.81 238.76))
+    (stroke (width 0) (type default))
+  )
   (wire (pts (xy 100.33 180.34) (xy 100.33 182.88))
     (stroke (width 0) (type default))
@@
     (stroke (width 0) (type default))
   )
+  (wire (pts (xy 257.81 233.68) (xy 257.81 238.76))
+    (stroke (width 0) (type default))
+  )
   (wire (pts (xy 135.255 87.63) (xy 153.67 87.63))
     (stroke (width 0) (type default))
@@
     (stroke (width 0) (type default))
   )
+  (wire (pts (xy 257.81 223.52) (xy 255.27 223.52))
+    (stroke (width 0) (type default))
+  )
   (wire (pts (xy 27.94 242.57) (xy 33.02 242.57))
     (stroke (width 0) (type default))
@@
     (stroke (width 0) (type default))
   )
+  (wire (pts (xy 255.27 228.6) (xy 257.81 228.6))
+    (stroke (width 0) (type default))
+  )
   (wire (pts (xy 153.67 87.63) (xy 153.67 90.17))
     (stroke (width 0) (type default))
@@
     )
   )
+  (symbol (lib_id "Connector_Generic:Conn_01x01") (at 250.19 233.68 180) (unit 1)
+    (in_bom yes) (on_board yes) (dnp no)
+    (property "Reference" "J9" (at 241.3 232.41 0)
+      (effects (font (size 1.27 1.27)))
+    )
+    (property "Value" "Conn_01x01" (at 241.3 234.95 0)
+      (effects (font (size 1.27 1.27)))
+    )
+    (property "Footprint" "Connector_PinHeader_2.54mm:PinHeader_1x01_P2.54mm_Vertical" (at 250.19 233.68 0)
+      (effects (font (size 1.27 1.27)) hide)
+    )
+    (property "Datasheet" "~" (at 250.19 233.68 0)
+      (effects (font (size 1.27 1.27)) hide)
+    )
+    (pin "1")
+    (instances
+      (project "AD5791 Linearity Calibrator"
+        (path "/545249ea-2c8e-4b30-8f2b-5f4518163292"
+          (reference "J9") (unit 1)
+        )
+      )
+    )
+  )
+  (symbol (lib_id "Connector_Generic:Conn_01x01") (at 250.19 228.6 180) (unit 1)
+    (in_bom yes) (on_board yes) (dnp no)
+    (property "Reference" "J8" (at 241.3 227.33 0)
+      (effects (font (size 1.27 1.27)))
+    )
+    (property "Value" "Conn_01x01" (at 241.3 229.87 0)
+      (effects (font (size 1.27 1.27)))
+    )
+    (property "Footprint" "Connector_PinHeader_2.54mm:PinHeader_1x01_P2.54mm_Vertical" (at 250.19 228.6 0)
+      (effects (font (size 1.27 1.27)) hide)
+    )
+    (property "Datasheet" "~" (at 250.19 228.6 0)
+      (effects (font (size 1.27 1.27)) hide)
+    )
+    (pin "1")
+    (instances
+      (project "AD5791 Linearity Calibrator"
+        (path "/545249ea-2c8e-4b30-8f2b-5f4518163292"
+          (reference "J8") (unit 1)
+        )
+      )
+    )
+  )
   (symbol (lib_id "Device:C_Small") (at 82.55 97.79 0) (unit 1)
     (in_bom yes) (on_board yes) (dnp no) (fields_autoplaced)
@@
     )
   )
+  (symbol (lib_id "power:GND") (at 257.81 241.3 0) (unit 1)
+    (in_bom yes) (on_board yes) (dnp no) (fields_autoplaced)
+    (property "Reference" "#PWR036" (at 257.81 247.65 0)
+      (effects (font (size 1.27 1.27)) hide)
+    )
+    (property "Value" "GND" (at 257.81 246.38 0)
+      (effects (font (size 1.27 1.27)))
+    )
+    (property "Footprint" "" (at 257.81 241.3 0)
+      (effects (font (size 1.27 1.27)) hide)
+    )
+    (property "Datasheet" "" (at 257.81 241.3 0)
+      (effects (font (size 1.27 1.27)) hide)
+    )
+    (pin "1")
+    (instances
+      (project "AD5791 Linearity Calibrator"
+        (path "/545249ea-2c8e-4b30-8f2b-5f4518163292"
+          (reference "#PWR036") (unit 1)
+        )
+      )
+      (project "TMP117 Breakout"
+        (path "/8e88e8ac-f1b3-4d96-ab24-388c44d4af4e"
+          (reference "#PWR04") (unit 1)
+        )
+      )
+    )
+  )
   (symbol (lib_id "Device:R") (at 72.39 63.5 180) (unit 1)
     (in_bom yes) (on_board yes) (dnp no)
@@
     )
   )
+  (symbol (lib_id "Connector_Generic:Conn_01x01") (at 250.19 223.52 180) (unit 1)
+    (in_bom yes) (on_board yes) (dnp no)
+    (property "Reference" "J7" (at 241.3 222.25 0)
+      (effects (font (size 1.27 1.27)))
+    )
+    (property "Value" "Conn_01x01" (at 241.3 224.79 0)
+      (effects (font (size 1.27 1.27)))
+    )
+    (property "Footprint" "Connector_PinHeader_2.54mm:PinHeader_1x01_P2.54mm_Vertical" (at 250.19 223.52 0)
+      (effects (font (size 1.27 1.27)) hide)
+    )
+    (property "Datasheet" "~" (at 250.19 223.52 0)
+      (effects (font (size 1.27 1.27)) hide)
+    )
+    (pin "1")
+    (instances
+      (project "AD5791 Linearity Calibrator"
+        (path "/545249ea-2c8e-4b30-8f2b-5f4518163292"
+          (reference "J7") (unit 1)
+        )
+      )
+    )
+  )
   (symbol (lib_id "power:+15V") (at 54.61 180.34 0) (unit 1)
     (in_bom yes) (on_board yes) (dnp no)
@@
         )
       )
+    )
+  )
+  (symbol (lib_id "Connector_Generic:Conn_01x01") (at 250.19 238.76 180) (unit 1)
+    (in_bom yes) (on_board yes) (dnp no)
+    (property "Reference" "J10" (at 241.3 237.49 0)
+      (effects (font (size 1.27 1.27)))
+    )
+    (property "Value" "Conn_01x01" (at 241.3 240.03 0)
+      (effects (font (size 1.27 1.27)))
+    )
+    (property "Footprint" "Connector_PinHeader_2.54mm:PinHeader_1x01_P2.54mm_Vertical" (at 250.19 238.76 0)
+      (effects (font (size 1.27 1.27)) hide)
+    )
+    (property "Datasheet" "~" (at 250.19 238.76 0)
+      (effects (font (size 1.27 1.27)) hide)
+    )
+    (pin "1")
+    (instances
+      (project "AD5791 Linearity Calibrator"
+        (path "/545249ea-2c8e-4b30-8f2b-5f4518163292"
+          (reference "J10") (unit 1)
+        )
+      )
